File: Pi HAT.kicad_sch (KiCad schematic)
At the start: 14 parts, among them J1 Screw_Terminal_01x04, J4 Barrel_Jack, J5 Screw_Terminal_01x03, J6 Screw_Terminal_01x03, J7 GPIO_CONNECTOR, Q1 S8550

Commit message: Minor tweaks on the board, board pullback, and 8550 error spotted
Other:
- note added: "Mistake on the 8550 footprint"
Changed lines of the file:
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@@
     (effects (font (size 2 2)) (justify left bottom))
+  )
+  (text "Mistake on the 8550 footprint" (at 87.63 21.59 0)
+    (effects (font (size 1.27 1.27)) (justify left bottom))
   )
   (text "Relay control" (at 147.955 52.07 0)
@@
       (effects (font (size 1.27 1.27)) hide)
     )
+    (pin "1")
+    (pin "2")
     (pin "3")
-    (pin "1")
-    (pin "2")
     (instances
       (project "Pi HAT"
@@
       (effects (font (size 1.27 1.27)) hide)
     )
+    (pin "1")
+    (pin "2")
     (pin "3")
-    (pin "1")
-    (pin "2")
     (instances
       (project "Pi HAT"
@@
       (effects (font (size 1.27 1.27)) hide)
     )
+    (pin "1")
+    (pin "2")
     (pin "3")
-    (pin "1")
-    (pin "2")
-    (instances
-      (project "Pi HAT"
+    (instances
+      (project "Pi HAT"

Commit message: Changed some of the wiring on the Jumpers, and changed the footprint for the 8550
Parts:
- removed Q1: S8550, Package_TO_SOT_SMD:SOT-23, symbol Transistor_BJT:S8550
- added Q1: S8550, Package_TO_SOT_SMD:SOT-23, symbol sensify:8550
Connections:
- net +5V: now also Q1.2 (E)
- net EXC+: now also JP12.1 (A); no longer JP12.2 (C)
- net INA+: now also JP9.1 (A); no longer JP9.2 (C)
- net INA-: now also JP11.1 (A); no longer JP11.2 (C)
- net LOAD_CELL_EXC: now also JP12.2 (C); no longer JP12.1 (A)
- net LOAD_CELL_PWR: now also Q1.3 (C)
- net S+: now also JP9.2 (C); no longer JP9.1 (A)
- net S-: now also JP11.2 (C); no longer JP11.1 (A)
- net at R1.1: now also Q1.1 (B)
Changed lines of the file:
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@@
     (stroke (width 0) (type default))
   )
-  (wire (pts (xy 140.462 128.524) (xy 155.194 128.524))
+  (wire (pts (xy 152.908 128.524) (xy 155.194 128.524))
     (stroke (width 0) (type default))
   )
@@
     (effects (font (size 1.27 1.27)) (justify left bottom))
   )
-  (label "LOAD_CELL_EXC" (at 140.462 128.524 0) (fields_autoplaced)
+  (label "LOAD_CELL_EXC" (at 168.656 132.334 0) (fields_autoplaced)
     (effects (font (size 1.27 1.27)) (justify left bottom))
   )
@@
     (effects (font (size 1.27 1.27)) (justify left bottom))
   )
-  (label "S-" (at 152.908 119.38 0) (fields_autoplaced)
+  (label "S-" (at 168.656 123.19 0) (fields_autoplaced)
     (effects (font (size 1.27 1.27)) (justify left bottom))
   )
@@
     (effects (font (size 1.27 1.27)) (justify left bottom))
   )
-  (label "S+" (at 152.4 109.728 0) (fields_autoplaced)
+  (label "S+" (at 168.656 113.538 0) (fields_autoplaced)
     (effects (font (size 1.27 1.27)) (justify left bottom))
   )
@@
     (effects (font (size 1.27 1.27)) (justify left bottom))
   )
-  (label "INA+" (at 168.656 113.538 180) (fields_autoplaced)
+  (label "INA+" (at 152.4 109.728 180) (fields_autoplaced)
     (effects (font (size 1.27 1.27)) (justify right bottom))
   )
@@
     (effects (font (size 1.27 1.27)) (justify left bottom))
   )
-  (label "INA-" (at 168.656 123.19 180) (fields_autoplaced)
+  (label "INA-" (at 152.908 119.38 180) (fields_autoplaced)
     (effects (font (size 1.27 1.27)) (justify right bottom))
   )
@@
     (effects (font (size 1.27 1.27)) (justify left bottom))
   )
-  (label "EXC+" (at 168.656 132.334 180) (fields_autoplaced)
+  (label "EXC+" (at 152.908 128.524 180) (fields_autoplaced)
     (effects (font (size 1.27 1.27)) (justify right bottom))
   )
@@
     )
   )
+  (symbol (lib_id "sensify:8550") (at 95.25 30.48 90) (unit 1)
+    (in_bom yes) (on_board yes) (dnp no)
+    (property "Reference" "Q1" (at 95.25 23.368 90)
+      (effects (font (size 1.27 1.27)))
+    )
+    (property "Value" "S8550" (at 95.25 25.908 90)
+      (effects (font (size 1.27 1.27)))
+    )
+    (property "Footprint" "Package_TO_SOT_SMD:SOT-23" (at 95.25 12.7 0)
+      (effects (font (size 1.27 1.27)) hide)
+    )
+    (property "Datasheet" "https://datasheet.lcsc.com/lcsc/2304140030_Jiangsu-Changjing-Electronics-Technology-Co---Ltd--S8550_C105432.pdf" (at 109.22 31.75 0)
+      (effects (font (size 1.27 1.27)) hide)
+    )
+    (pin "1")
+    (pin "2")
+    (pin "3")
+    (instances
+      (project "Pi HAT"
+        (path "/48f827a8-6e22-4a2e-abdc-c2a03098d883"
+          (reference "Q1") (unit 1)
+        )
+      )
+      (project "flexo"
+        (path "/4e8f7957-453a-4cfe-b48f-8c226e41d404/f6d346dd-8575-47bd-8687-3a3372179ec2"
+          (reference "Q6") (unit 1)
+        )
+      )
+    )
+  )
   (symbol (lib_name "+5V_1") (lib_id "power:+5V") (at 179.07 24.13 0) (unit 1)
     (in_bom yes) (on_board yes) (dnp no)
@@
         )
       )
-    )
-  )
-  (symbol (lib_id "Transistor_BJT:S8550") (at 95.25 33.02 270) (mirror x) (unit 1)
-    (in_bom yes) (on_board yes) (dnp no) (fields_autoplaced)
-    (property "Reference" "Q1" (at 95.25 24.13 90)
-      (effects (font (size 1.27 1.27)))
-    )
-    (property "Value" "S8550" (at 95.25 26.67 90)
-      (effects (font (size 1.27 1.27)))
-    )
-    (property "Footprint" "Package_TO_SOT_SMD:SOT-23" (at 93.345 27.94 0)
-      (effects (font (size 1.27 1.27) italic) (justify left) hide)
-    )
-    (property "Datasheet" "http://www.unisonic.com.tw/datasheet/S8550.pdf" (at 95.25 33.02 0)
-      (effects (font (size 1.27 1.27)) (justify left) hide)
-    )
-    (property "Populate" "1" (at 95.25 33.02 0)
-      (effects (font (size 1.27 1.27)) hide)
-    )
-    (property "Extended" "0" (at 95.25 33.02 0)
-      (effects (font (size 1.27 1.27)) hide)
-    )
-    (property "LCSC" "C8542" (at 95.25 33.02 0)
-      (effects (font (size 1.27 1.27)) hide)
-    )
-    (pin "1")
-    (pin "2")
-    (pin "3")
-    (instances
-      (project "Pi HAT"
-        (path "/48f827a8-6e22-4a2e-abdc-c2a03098d883"
-          (reference "Q1") (unit 1)
-        )
-      )
