File: hx711.kicad_sch (KiCad schematic)
At the start: 16 parts, among them Q4 S8550, U6 HX711

Commit message: Added footprints for HX711 circuit on PCB and modified pin assignment
Parts:
- C18, C22, C23: footprint (none) -> Capacitor_SMD:C_0603_1608Metric
- C19, C20, C21, C24: footprint (none) -> Capacitor_SMD:C_0402_1005Metric
- JP10: footprint (none) -> Jumper:SolderJumper-2_P1.3mm_Bridged_Pad1.0x1.5mm
- L1: footprint (none) -> Inductor_SMD:L_0603_1608Metric
- Q4: footprint Package_TO_SOT_THT:TO-92_Inline -> Package_TO_SOT_SMD:SOT-23
- R18, R19, R20, R21, R22: footprint (none) -> Resistor_SMD:R_0402_1005Metric
Changed lines of the file:
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@@
       (effects (font (size 1.27 1.27)) (justify left))
     )
-    (property "Footprint" "" (at 103.124 77.978 0)
+    (property "Footprint" "Capacitor_SMD:C_0603_1608Metric" (at 103.124 77.978 0)
       (effects (font (size 1.27 1.27)) hide)
     )
@@
       (effects (font (size 1.27 1.27)) (justify left))
     )
-    (property "Footprint" "" (at 128.27 92.71 0)
+    (property "Footprint" "Capacitor_SMD:C_0402_1005Metric" (at 128.27 92.71 0)
       (effects (font (size 1.27 1.27)) hide)
     )
@@
       (effects (font (size 1.27 1.27)) (justify left))
     )
-    (property "Footprint" "" (at 116.84 98.806 0)
+    (property "Footprint" "Resistor_SMD:R_0402_1005Metric" (at 116.84 98.806 0)
       (effects (font (size 1.27 1.27)) hide)
     )
@@
       (effects (font (size 1.27 1.27)) (justify left))
     )
-    (property "Footprint" "Package_TO_SOT_THT:TO-92_Inline" (at 132.715 64.77 0)
+    (property "Footprint" "Package_TO_SOT_SMD:SOT-23" (at 132.715 64.77 0)
       (effects (font (size 1.27 1.27) italic) (justify left) hide)
     )
@@
       (effects (font (size 1.27 1.27)) (justify left))
     )
-    (property "Footprint" "" (at 119.38 98.806 0)
+    (property "Footprint" "Resistor_SMD:R_0402_1005Metric" (at 119.38 98.806 0)
       (effects (font (size 1.27 1.27)) hide)
     )
@@
       (effects (font (size 1.27 1.27)))
     )
-    (property "Footprint" "" (at 162.56 101.6 0)
+    (property "Footprint" "Jumper:SolderJumper-2_P1.3mm_Bridged_Pad1.0x1.5mm" (at 162.56 101.6 0)
       (effects (font (size 1.27 1.27)) hide)
     )
@@
       (effects (font (size 1.27 1.27)))
     )
-    (property "Footprint" "" (at 115.824 74.422 0)
+    (property "Footprint" "Inductor_SMD:L_0603_1608Metric" (at 115.824 74.422 0)
       (effects (font (size 1.27 1.27)) hide)
     )
@@
       (effects (font (size 1.27 1.27)) (justify left))
     )
-    (property "Footprint" "" (at 185.166 66.04 0)
+    (property "Footprint" "Capacitor_SMD:C_0603_1608Metric" (at 185.166 66.04 0)
       (effects (font (size 1.27 1.27)) hide)
     )
@@
       (effects (font (size 1.27 1.27)) (justify left))
     )
-    (property "Footprint" "" (at 125.73 80.01 0)
+    (property "Footprint" "Resistor_SMD:R_0402_1005Metric" (at 125.73 80.01 0)
       (effects (font (size 1.27 1.27)) hide)
     )
@@
       (effects (font (size 1.27 1.27)) (justify left))
     )
-    (property "Footprint" "" (at 118.11 83.82 0)
+    (property "Footprint" "Resistor_SMD:R_0402_1005Metric" (at 118.11 83.82 0)
       (effects (font (size 1.27 1.27)) hide)
     )
@@
       (effects (font (size 1.27 1.27)) (justify left))
     )
-    (property "Footprint" "" (at 190.246 66.04 0)
+    (property "Footprint" "Capacitor_SMD:C_0402_1005Metric" (at 190.246 66.04 0)
       (effects (font (size 1.27 1.27)) hide)
     )
@@
       (effects (font (size 1.27 1.27)) (justify left))
     )
-    (property "Footprint" "" (at 174.498 66.04 0)
+    (property "Footprint" "Capacitor_SMD:C_0402_1005Metric" (at 174.498 66.04 0)
       (effects (font (size 1.27 1.27)) hide)
     )
@@
       (effects (font (size 1.27 1.27)) (justify left))
     )
-    (property "Footprint" "" (at 107.442 77.978 0)
+    (property "Footprint" "Capacitor_SMD:C_0603_1608Metric" (at 107.442 77.978 0)
       (effects (font (size 1.27 1.27)) hide)
     )
@@
       (effects (font (size 1.27 1.27)) (justify left))
     )
-    (property "Footprint" "" (at 128.27 110.49 0)
+    (property "Footprint" "Capacitor_SMD:C_0402_1005Metric" (at 128.27 110.49 0)
       (effects (font (size 1.27 1.27)) hide)
     )
@@
       (effects (font (size 1.27 1.27)) (justify left))
     )
-    (property "Footprint" "" (at 157.48 105.918 0)
-      (effects (font (size 1.27 1.27)) hide)
-    )
+    (property "Footprint" "Resistor_SMD:R_0402_1005Metric" (at 157.48 105.918 0)
+      (effects (font (size 1.27 1.27)) hide)
+    )

Commit message: Fixed HX711 decoupling cap. Changed EXC+.
- Changed EXC+ to 4.06V
- Consistent values for schematic components
- Added B.silkscreen art
Parts:
- C19, C21, C24: value 100nF -> 100n
- C22: value 10uF -> 10u
- C23: value 10uF -> 100n
- R18: value 33k -> 27k
Other:
- note added: "(VFB=1.25V)"
- note added: "AVDD = VFB(R1+R2)/R2 = 4.06V"
- note added: "R1"
- note added: "R2"
- note removed: "(VBG=1.25V)"
- note removed: "AVDD = VBG(R1+R2)/R2 = 4.69V"
Changed lines of the file:
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@@
     (stroke (width 0) (type default))
+  )
+  (text "R1" (at 118.11 80.772 0)
+    (effects (font (size 1.27 1.27)) (justify left bottom))
   )
   (text "Default 10SPS ODR\nBreak off jumper to set 80SPS ODR"
@@
     (effects (font (size 1.27 1.27)) (justify left bottom))
   )
-  (text "AVDD = VBG(R1+R2)/R2\n	 = 4.69V" (at 82.042 92.202 0)
+  (text "AVDD = VFB(R1+R2)/R2\n	 = 4.06V" (at 82.042 92.202 0)
     (effects (font (size 1.27 1.27)) (justify left bottom))
   )
-  (text "(VBG=1.25V)" (at 81.788 94.742 0)
+  (text "(VFB=1.25V)" (at 81.788 94.742 0)
+    (effects (font (size 1.27 1.27)) (justify left bottom))
+  )
+  (text "R2" (at 114.046 83.566 0)
     (effects (font (size 1.27 1.27)) (justify left bottom))
   )
@@
       (effects (font (size 1.27 1.27)) (justify left))
     )
-    (property "Value" "10uF" (at 100.584 78.232 0)
+    (property "Value" "100n" (at 100.584 78.232 0)
       (effects (font (size 1.27 1.27)) (justify left))
     )
@@
       (effects (font (size 1.27 1.27)) (justify left))
     )
-    (property "Value" "10uF" (at 182.626 67.3163 0)
+    (property "Value" "10u" (at 182.626 67.3163 0)
       (effects (font (size 1.27 1.27)) (justify left))
     )
@@
       (effects (font (size 1.27 1.27)) (justify left))
     )
-    (property "Value" "33k" (at 124.46 80.518 0)
+    (property "Value" "27k" (at 124.46 80.518 0)
       (effects (font (size 1.27 1.27)) (justify left))
     )
@@
       (effects (font (size 1.27 1.27)) (justify left))
     )
-    (property "Value" "100nF" (at 192.786 67.3163 0)
+    (property "Value" "100n" (at 192.786 67.3163 0)
       (effects (font (size 1.27 1.27)) (justify left))
     )
@@
       (effects (font (size 1.27 1.27)) (justify left))
     )
-    (property "Value" "100nF" (at 171.958 67.3163 0)
+    (property "Value" "100n" (at 171.958 67.3163 0)
       (effects (font (size 1.27 1.27)) (justify left))
     )
@@
       (effects (font (size 1.27 1.27)) (justify left))
     )
-    (property "Value" "100nF" (at 126.238 111.76 0)
-      (effects (font (size 1.27 1.27)) (justify left))
-    )
+    (property "Value" "100n" (at 126.238 111.76 0)
+      (effects (font (size 1.27 1.27)) (justify left))
+    )

Commit message: Fixed JP10 jumper footprint
Parts:
- JP10: footprint Jumper:SolderJumper-2_P1.3mm_Bridged_Pad1.0x1.5mm -> Jumper:SolderJumper-2_P1.3mm_Bridged_RoundedPad1.0x1.5mm
Changed lines of the file:
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@@
       (effects (font (size 1.27 1.27)))
     )
-    (property "Footprint" "Jumper:SolderJumper-2_P1.3mm_Bridged_Pad1.0x1.5mm" (at 162.56 101.6 0)
+    (property "Footprint" "Jumper:SolderJumper-2_P1.3mm_Bridged_RoundedPad1.0x1.5mm" (at 162.56 101.6 0)
       (effects (font (size 1.27 1.27)) hide)
     )

Commit message: Added jlcpcb files. Updated additional libraries
Parts:
- C18: value 10uF -> 10u
- C20: value 100nF -> 100n
Changed lines of the file:
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@@
       (effects (font (size 1.27 1.27)) (justify left))
     )
-    (property "Value" "100nF" (at 132.08 88.646 0)
+    (property "Value" "100n" (at 132.08 88.646 0)
       (effects (font (size 1.27 1.27)) (justify left))
     )
@@
       (effects (font (size 1.27 1.27)) (justify left))
     )
-    (property "Value" "10uF" (at 109.982 78.232 0)
-      (effects (font (size 1.27 1.27)) (justify left))
-    )
+    (property "Value" "10u" (at 109.982 78.232 0)
+      (effects (font (size 1.27 1.27)) (justify left))
+    )

Commit message: Minor tweaks on the board, board pullback, and 8550 error spotted
Other:
- note added: "Mistake on the 8550 footprint"
Changed lines of the file:
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@@
+    (effects (font (size 1.27 1.27)) (justify left bottom))
+  )
+  (text "Mistake on the 8550 footprint" (at 116.205 57.15 0)
     (effects (font (size 1.27 1.27)) (justify left bottom))
   )
@@
       (effects (font (size 1.27 1.27)) (justify left) hide)
     )
+    (pin "1")
+    (pin "2")
     (pin "3")
-    (pin "1")
-    (pin "2")
     (instances
       (project "Pi HAT"
@@
       (effects (font (size 1.27 1.27)) hide)
     )
-    (pin "2")
-    (pin "1")
+    (pin "1")
+    (pin "2")
     (instances
       (project "Pi HAT"
@@
       (effects (font (size 1.27 1.27)) hide)
     )
+    (pin "1")
     (pin "10")
+    (pin "11")
+    (pin "12")
+    (pin "13")
     (pin "14")
+    (pin "15")
+    (pin "16")
+    (pin "2")
+    (pin "3")
+    (pin "4")
+    (pin "5")
+    (pin "6")
     (pin "7")
-    (pin "16")
-    (pin "4")
-    (pin "13")
-    (pin "1")
-    (pin "2")
-    (pin "6")
     (pin "8")
     (pin "9")
-    (pin "3")
-    (pin "15")
-    (pin "5")
-    (pin "11")
-    (pin "12")
-    (instances
-      (project "Pi HAT"
+    (instances
+      (project "Pi HAT"

Commit message: Changed some of the wiring on the Jumpers, and changed the footprint for the 8550
Parts:
- removed Q4: S8550, Package_TO_SOT_SMD:SOT-23, symbol Transistor_BJT:S8550
- added Q1: S8550, Package_TO_SOT_SMD:SOT-23, symbol sensify:8550
Connections:
- net VCC: now also Q1.2 (E)
- net at U6.2 (BASE): now also Q1.1 (B)
- net at L1.2, R18.1, U6.3 (AVDD): now also Q1.3 (C)
Changed lines of the file:
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@@
-    )
-  )
-  (symbol (lib_id "Transistor_BJT:S8550") (at 130.81 69.85 90) (unit 1)
-    (in_bom yes) (on_board yes) (dnp no)
-    (property "Reference" "Q4" (at 132.08 64.77 0)
-      (effects (font (size 1.27 1.27)) (justify left))
-    )
-    (property "Value" "S8550" (at 129.54 64.77 0)
-      (effects (font (size 1.27 1.27)) (justify left))
-    )
-    (property "Footprint" "Package_TO_SOT_SMD:SOT-23" (at 132.715 64.77 0)
-      (effects (font (size 1.27 1.27) italic) (justify left) hide)
-    )
-    (property "Datasheet" "http://www.unisonic.com.tw/datasheet/S8550.pdf" (at 130.81 69.85 0)
-      (effects (font (size 1.27 1.27)) (justify left) hide)
-    )
-    (pin "1")
-    (pin "2")
-    (pin "3")
-    (instances
-      (project "Pi HAT"
-        (path "/48f827a8-6e22-4a2e-abdc-c2a03098d883/dad399bb-460b-4f5e-b266-a80a3ab180e2"
-          (reference "Q4") (unit 1)
-        )
-      )
     )
   )
@@
         )
       )
+    )
+  )
+  (symbol (lib_id "sensify:8550") (at 130.81 67.31 270) (mirror x) (unit 1)
+    (in_bom yes) (on_board yes) (dnp no)
+    (property "Reference" "Q1" (at 130.81 60.198 90)
+      (effects (font (size 1.27 1.27)))
+    )
+    (property "Value" "S8550" (at 130.81 62.738 90)
+      (effects (font (size 1.27 1.27)))
+    )
+    (property "Footprint" "Package_TO_SOT_SMD:SOT-23" (at 130.81 49.53 0)
+      (effects (font (size 1.27 1.27)) hide)
+    )
+    (property "Datasheet" "https://datasheet.lcsc.com/lcsc/2304140030_Jiangsu-Changjing-Electronics-Technology-Co---Ltd--S8550_C105432.pdf" (at 116.84 68.58 0)
+      (effects (font (size 1.27 1.27)) hide)
+    )
+    (pin "1")
+    (pin "2")
+    (pin "3")
+    (instances
+      (project "Pi HAT"
+        (path "/48f827a8-6e22-4a2e-abdc-c2a03098d883"
+          (reference "Q1") (unit 1)
+        )
+        (path "/48f827a8-6e22-4a2e-abdc-c2a03098d883/dad399bb-460b-4f5e-b266-a80a3ab180e2"
+          (reference "Q4") (unit 1)
+        )
+      )
+      (project "flexo"
+        (path "/4e8f7957-453a-4cfe-b48f-8c226e41d404/f6d346dd-8575-47bd-8687-3a3372179ec2"
+          (reference "Q6") (unit 1)
+        )
+      )
