File: amp_sch.kicad_sch (KiCad schematic)
At the start: 15 parts, among them IC1 AD7730, U1 74LVC125APW,118

Commit message: Connected NO2 to COM1. Annonated relays.
Other:
- title: (none) -> Raspberry Pi Zero Intrumentation HAT
Changed lines of the file:
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@@
   (paper "A4")
   (title_block
-    (rev "1.2.0")
+    (title "Raspberry Pi Zero Intrumentation HAT")
+    (date "2024-06-07")
+    (rev "1.3.0")
+    (comment 1 "@supervisor Justin Pead")
+    (comment 2 "@author Montso Mokake")
   )
   (junction (at 180.34 90.17) (diameter 0) (color 0 0 0 0)

Commit message: Ammended it to have the jumper connection
Parts:
- renumbered JP6 to JP8
