File: power_monitor.kicad_sch (KiCad schematic)
At the start: 28 parts, among them J11 Conn_01x02_Male, J9 Conn_01x03_Male, U2 CJ431, U3 TMP23X, U4 ACS712x, U5 ADC108S022CIMTX

Commit message: Update BJT symbols and ver number
Parts:
- removed U2: CJ431, Package_TO_SOT_SMD:SOT-23, symbol Reference_Voltage:CJ432
Changed lines of the file:
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@@
     (title "Power Monitor")
     (date "2022-12-18")
-    (rev "1.1.0")
+    (rev "1.2.0")
     (comment 1 "@author Montso Mokake ")
     (comment 2 "@reference Pi_ADC/Justin Pead")
@@
   )
   (junction (at 39.37 184.15) (diameter 0) (color 0 0 0 0)
-  )
-  (junction (at 39.37 176.53) (diameter 0) (color 0 0 0 0)
   )
   (junction (at 252.476 105.156) (diameter 0) (color 0 0 0 0)
@@
         )
       )
-    )
-  )
-  (symbol (lib_id "Reference_Voltage:CJ432") (at 39.37 179.07 270) (mirror x) (unit 1)
-    (in_bom yes) (on_board yes) (dnp no)
-    (property "Reference" "U2" (at 36.83 181.3814 90)
-      (effects (font (size 1.27 1.27)) (justify right))
-    )
-    (property "Value" "CJ431" (at 36.83 179.07 90)
-      (effects (font (size 1.27 1.27)) (justify right))
-    )
-    (property "Footprint" "Package_TO_SOT_SMD:SOT-23" (at 35.56 179.07 0)
-      (effects (font (size 1.27 1.27) italic) hide)
-    )
-    (property "Datasheet" "http://www.cj-elec.com/txUpfile/20134181474991806.pdf" (at 39.37 179.07 0)
-      (effects (font (size 1.27 1.27) italic) hide)
-    )
-    (property "Extended" "0" (at 39.37 179.07 0)
-      (effects (font (size 1.27 1.27)) hide)
-    )
-    (property "LCSC" "C3113" (at 39.37 179.07 0)
-      (effects (font (size 1.27 1.27)) hide)
-    )
-    (property "Populate" "1" (at 39.37 179.07 0)
-      (effects (font (size 1.27 1.27)) hide)
-    )
-    (property "Price" "0.04" (at 39.37 179.07 0)
-      (effects (font (size 1.27 1.27)) hide)
-    )
-    (pin "1")
-    (pin "2")
-    (pin "3")
-    (instances
-      (project "Pi HAT"
-        (path "/48f827a8-6e22-4a2e-abdc-c2a03098d883/715798e8-ada1-4b31-bdfe-4378c151d2b8"
-          (reference "U2") (unit 1)
-        )
-      )

Commit message: Connected NO2 to COM1. Annonated relays.
Other:
- title: Power Monitor -> Raspberry Pi Zero Intrumentation HAT
Changed lines of the file:
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@@
   (paper "A4")
   (title_block
-    (title "Power Monitor")
-    (date "2022-12-18")
-    (rev "1.2.0")
-    (comment 1 "@author Montso Mokake ")
-    (comment 2 "@reference Pi_ADC/Justin Pead")
+    (title "Raspberry Pi Zero Intrumentation HAT")
+    (date "2024-06-07")
+    (rev "1.3.0")
+    (comment 1 "@supervisor Justin Pead")
+    (comment 2 "@author Montso Mokake")
   )
   (junction (at 115.316 93.218) (diameter 0) (color 0 0 0 0)
